File: AudioPlug2SMA_M1V1/AudioPlug2SMA_M1V1.kicad_pcb (KiCad board)
At the start: 2 copper layers, 21.6 x 33 mm, 7 parts, among them J1 SMA-KHD105, J2 SMA-KHD105, J3 SP-3533-02

Commit message: Update AudioPlug2SMA_M1V1
Parts:
- removed the REF** at (100.3, 115.6)
- removed the REF** at (83.8, 115.6)
- removed the REF** at (100.3, 87.6)
- removed the REF** at (83.8, 87.6)
- added REF**: MountingHole_2.2mm_M2_Pad, MountingHole:MountingHole_2.2mm_M2_Pad, F.Cu at (83.8, 87.6)
- added REF**: MountingHole_2.2mm_M2_Pad, MountingHole:MountingHole_2.2mm_M2_Pad, F.Cu at (100.3, 115.6)
- added REF**: MountingHole_2.2mm_M2_Pad, MountingHole:MountingHole_2.2mm_M2_Pad, F.Cu at (83.8, 115.6)
- added REF**: MountingHole_2.2mm_M2_Pad, MountingHole:MountingHole_2.2mm_M2_Pad, F.Cu at (100.3, 87.6)
Routing:
- net GNDREF: vias 195 -> 156
